File: LCD7th.kicad_pcb (KiCad board)
At the start: 2 copper layers, 51.5 x 100 mm, 61 parts, among them P1 USB_B, P2 BATT, P3 ICSP, P4 UART, P5 I2C, P6 5VCONN, P7 BATT, Q1 2N7002, SW1 SW1, SW2 SW2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

Commit message: update
Parts:
- removed Q1: 2N7002, TO_SOT_Packages_SMD:SOT-23
- added C21: 100nF, Capacitors_SMD:C_0805_HandSoldering, F.Cu at (81.2, 68.0)
- added P8: BATT, LCD7th:CR2477, F.Cu at (43.7, 123.9)
- added R11: 1K, Resistors_SMD:R_0805_HandSoldering, F.Cu at (81.2, 56.8)
- added R12: 1K, Resistors_SMD:R_0805_HandSoldering, F.Cu at (81.2, 58.8)
- added SW7: BG_POWER, Buttons_Switches_SMD:SW_SPDT_PCM12, F.Cu at (43.0, 87.8)
- C1: value 4.7uF -> 0.1uF
- C4: value 0.1uF -> 4.7uF
- R1, R10: value 470R -> 1K
- R9: value 220R -> 330R
- moved R8 32.6 mm to (81.2, 54.8)
- moved C9 6.81 mm to (81.2, 62.0)
- moved C3 4.59 mm to (81.2, 66.0), turned to 180 degrees
- moved C2 4.08 mm to (81.2, 64.0), turned to 180 degrees
- moved R9 2.21 mm to (49.7, 46.0)
- moved R2 2.09 mm to (74.2, 135.6)
- moved R3 2.09 mm to (74.2, 137.6)
- moved R5 0.57 mm to (81.2, 52.8)
Connections:
- C1 pad 1: +5C -> +3V3
- C4 pad 1: +3V3 -> +5C
- D1 pad 1: +5C -> Net-(D1-Pad1)
- D4 pad 2: +3V3 -> Net-(D4-Pad2)
- R8 pad 1: /BLED -> +5C
- R9 pad 2: Net-(Q1-Pad3) -> GND
- SW5 pad 1: GND -> Net-(SW5-Pad1)
- SW5 pad 2: Net-(SW5-Pad2) -> +5C
- SW5 pad 3: +5C -> Net-(D1-Pad1)
- U2 pad 3: Net-(SW5-Pad2) -> +5C
- U3 pad 30: /BLED -> /BATADC
Routing:
- net Net-(D4-Pad2): track 0.00 -> 44.5 mm
- net /BATADC: track 0.00 -> 35.9 mm, vias 0 -> 2
- net Net-(C16-Pad2): track 42.9 -> 20.0 mm
- net /BLED: track 20.7 -> 0.00 mm
- net Net-(D1-Pad1): track 0.00 -> 18.4 mm
- net +BATT: track 56.0 -> 74.2 mm, vias 0 -> 1
- net Net-(LCD1-Pad4): track 35.9 -> 18.7 mm
- net Net-(SW5-Pad2): track 17.0 -> 0.00 mm
- net +5C: track 134.6 -> 150.1 mm, vias 0 -> 1
- net /D-: track 76.7 -> 91.7 mm
- net Net-(C19-Pad1): track 27.6 -> 15.0 mm, vias 0 -> 2
- net /D+: track 80.5 -> 91.7 mm
- net Net-(LCD1-Pad6): track 19.9 -> 10.6 mm, vias 0 -> 2
- net GND: track 486.2 -> 478.4 mm, vias 16 -> 9
- net Net-(P3-Pad5): track 38.3 -> 31.9 mm, vias 1 -> 0
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Other:
- outline, holes or cut-outs redrawn
- board text added: "LCD7th V1.1"
