File: LCD7th.sch (KiCad schematic (older format))
At the start: 56 parts, among them P1 USB_B, P2 BATT, P3 ICSP, P4 UART, P5 I2C, P6 5VCONN, P7 BATT, Q1 2N7002, SW1 SW1, SW2 SW2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

Commit message: update
Parts:
- removed Q1: 2N7002, TO_SOT_Packages_SMD:SOT-23, symbol 2N7002
- removed R8: 1K, Resistors_SMD:R_0805_HandSoldering, symbol R_Small
- added C21: 100nF, Capacitors_SMD:C_0805_HandSoldering, symbol C_Small
- added P8: BATT, LCD7th:LiConn, symbol CONN_01X02
- added R12: 1K, Resistors_SMD:R_0805_HandSoldering, symbol R_Small
- added SW7: BG_POWER, Buttons_Switches_SMD:SW_SPDT_PCM12, symbol Switch_SPDT_x2
- D2, D3, D4, LED1, LED2: symbol LED -> LED-RESCUE-LCD7th
- P1: symbol USB_B -> USB_B-RESCUE-LCD7th
- R1, R10: value 470R -> 1K
- R9: value 220R -> 330R
- U3: symbol ATmega32U4-AU -> ATmega32U4-AU-RESCUE-LCD7th
- renumbered C2 to C1, C3 to C2, C4 to C3, C1 to C4
Connections:
- net labels added: BATADC
- net labels removed: BLED
- wire segments 239 -> 242
- no-connect marks 5 -> 7
Other:
- moved on the sheet: C10, D2, D3, D4, R6, R7, R9, U2
