File: hardware/_autosave-LCD7th.kicad_pcb (KiCad board)
At the start: 2 copper layers, 51.5 x 100 mm, 58 parts, among them P1 USB_B, P2 BATT, P3 ICSP, P4 UART, P5 I2C, P6 5VCONN, P7 BATT, P8 BATT, SW1 SW1, SW2 SW2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

Commit message: update
Parts:
- added G***: LOGO, LCD7th:szdiy_logo, F.Cu at (102.8, 92.6)
- moved P3 82.0 mm to (44.2, 120.7)
- moved C1 49.8 mm to (59.0, 86.7)
- moved LED1 43.0 mm to (62.9, 101.3)
- moved R1 42.7 mm to (62.9, 97.3)
- moved LED2 41.8 mm to (67.3, 101.3)
- moved R10 41.3 mm to (67.3, 97.3)
- moved U1 41.0 mm to (65.9, 92.1)
- moved SW7 40.7 mm to (43.4, 47.0)
- moved R4 39.8 mm to (50.9, 96.7), turned to 270 degrees
- moved C5 39.6 mm to (55.5, 96.7)
- moved P7 36.5 mm to (80.5, 137.3)
- moved P1 35.4 mm to (46.2, 137.4)
- moved C4 35.0 mm to (51.7, 86.6)
- moved D1 33.5 mm to (71.1, 91.8), turned to 0 degrees
- moved C6 33.4 mm to (55.6, 86.7)
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Other:
- board size 51.5 x 100 mm -> 48 x 100 mm
- board text removed: "-"
- board text removed: "G"
- board text removed: "R"
- board text removed: "SZDIY 2009-2016"
- board text removed: "SZDIY.ORG"
- board text removed: "Y"
