File: hardware/LCD7th.kicad_pcb (KiCad board)
At the start: 2 copper layers, 51.5 x 100 mm, 65 parts, among them P1 USB_B, P2 BATT, P3 ICSP, P4 UART, P5 I2C, P6 5VCONN, P7 BATT, P8 BATT, SW1 SW1, SW2 SW2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

Commit message: update
Parts:
- removed MH1, MH2, MH3: MountingHole_3.2mm_M3_ISO14580_Pad, Mounting_Holes:MountingHole_3.2mm_M3_ISO14580_Pad
- removed PT1: prototyping, LCD7th:prototyping
- removed R11, R8: 1K, Resistors_SMD:R_0805_HandSoldering
- removed REF**: Symbol_GNU-Logo_SilkscreenTop, Symbols:Symbol_GNU-Logo_SilkscreenTop
- C1, C10, C11, C12, C13, C14, C15, C16, C17, C18, C19, C2, C20, C21, C3, C4, C5, C6, C7, C8, C9: footprint Capacitors_SMD:C_0805_HandSoldering -> Capacitors_SMD:C_0603_HandSoldering
- D1: value B340A -> M7; footprint LCD7th:B340A -> LCD7th:DIODE_DO214AC-SMA
- D2, D3, LED1, LED2: footprint LEDs:LED_0805 -> LEDs:LED_0603
- D4: footprint Pin_Headers:Pin_Header_Straight_1x02 -> LEDs:LED_0603
- P8: footprint LCD7th:CR2477 -> SmartEye:CR2477_s
- R1, R10, R12, R2, R3, R4, R5, R6, R7, R9: footprint Resistors_SMD:R_0805_HandSoldering -> Resistors_SMD:R_0603_HandSoldering
- SP1: footprint LCD7th:TAT-BP1109S -> Buzzers_Beepers:BUZZER
- SW1, SW2, SW3, SW4, SW6: footprint Buttons_Switches_SMD:SW_SPST_EVQQ2 -> Buttons_Switches_SMD:SW_SPST_EVPBF
- X1: footprint Crystals:Crystal_SMD_5032_4Pads -> Crystals:crystal_FA238-TSX3225
- moved P3 82.0 mm to (44.2, 120.7)
- moved C1 49.8 mm to (59.0, 86.7)
- moved LED1 43.0 mm to (62.9, 101.3)
- moved R1 42.7 mm to (62.9, 97.3)
- moved LED2 41.8 mm to (67.3, 101.3)
- moved R10 41.3 mm to (67.3, 97.3)
- moved U1 41.0 mm to (65.9, 92.1)
- moved SW7 40.8 mm to (43.4, 47.0)
- moved R4 39.8 mm to (50.9, 96.7), turned to 270 degrees
- moved C5 39.6 mm to (55.5, 96.7)
- moved SP1 37.1 mm to (48.0, 110.0)
- moved P1 35.4 mm to (46.2, 137.4)
- moved C4 35.0 mm to (51.7, 86.6)
- moved D1 33.5 mm to (71.1, 91.8), turned to 0 degrees
- moved C6 33.4 mm to (55.6, 86.7)
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Connections:
- D1 pad 1: Net-(D1-Pad1) -> +5C
- LCD1 pad 0: Net-(LCD1-Pad0) -> (no net)
- LCD1 pad 28: Net-(LCD1-Pad28) -> (no net)
- P2 pad 2: +BATT -> Net-(P2-Pad2)
- P7 pad 2: +BATT -> Net-(P2-Pad2)
- P8 pad 2: +BATT -> Net-(P2-Pad2)
- R12 pad 2: Net-(R11-Pad1) -> +BATT
- SW5 pad 1: Net-(SW5-Pad1) -> +BATT
- SW5 pad 2: +5C -> Net-(P2-Pad2)
- SW5 pad 3: Net-(D1-Pad1) -> (no net)
- SW7 pad 3: Net-(SW7-Pad3) -> (no net)
- U3 pad 2: Net-(U3-Pad2) -> (no net)
Routing:
- net GND: track 478.4 -> 0.00 mm, vias 9 -> 0
- net +3V3: track 224.7 -> 0.00 mm, vias 1 -> 0
- net +5C: track 150.1 -> 0.00 mm, vias 1 -> 0
- net /MOSI: track 115.3 -> 0.00 mm, vias 1 -> 0
- net /MISO: track 110.0 -> 0.00 mm, vias 1 -> 0
- net /SCK: track 104.8 -> 0.00 mm, vias 1 -> 0
- net /D-: track 91.7 -> 0.00 mm
- net /D+: track 91.7 -> 0.00 mm
- net +BATT: track 74.2 -> 0.00 mm, vias 1 -> 0
- net Net-(SW4-Pad1): track 69.9 -> 0.00 mm, vias 1 -> 0
- net Net-(D4-Pad2): track 44.5 -> 0.00 mm
- net /SCL: track 44.3 -> 0.00 mm, vias 1 -> 0
- net /SDA: track 42.5 -> 0.00 mm, vias 1 -> 0
- net /BATADC: track 35.9 -> 0.00 mm, vias 2 -> 0
- net /BUZZER: track 32.7 -> 0.00 mm, vias 2 -> 0
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- removed copper zone on B.Cu, net GND
- removed copper zone on F.Cu, net GND
Other:
- board size 51.5 x 100 mm -> 48 x 100 mm
- board text removed: "-"
- board text removed: "G"
- board text removed: "R"
- board text removed: "SZDIY 2009-2016"
- board text removed: "SZDIY COMMUNITY 2009.4.19-2016.4.19"
- board text removed: "SZDIY.ORG"
- board text removed: "Y"

Commit message: uppdate layout
Parts:
- added G***: LOGO, LCD7th:szdiy_logo, F.Cu at (69.2, 99.8)
- D4: footprint LEDs:LED_0603 -> Connectors:CONN_2.54mm_1x2
- P4, P5: footprint Pin_Headers:Pin_Header_Straight_1x04 -> Connectors:CONN_2.54mm_1x4
- P6: footprint Pin_Headers:Pin_Header_Straight_1x02 -> Connectors:CONN_2.54mm_1x2
- moved C4 44.8 mm to (49.1, 131.3)
- moved SW7 41.4 mm to (84.8, 46.8), turned to 90 degrees
- moved C6 37.8 mm to (80.4, 58.2), turned to 180 degrees
- moved C1 37.3 mm to (80.4, 56.2), turned to 180 degrees
- moved R12 35.8 mm to (58.0, 85.4), turned to 270 degrees
- moved SW6 32.8 mm to (47.6, 45.7), turned to 0 degrees
- moved R9 31.9 mm to (80.5, 54.2)
- moved D4 29.3 mm to (78.8, 45.9), turned to 270 degrees
- moved R5 26.4 mm to (53.8, 46.0), turned to 270 degrees
- moved R1 19.4 mm to (44.2, 92.0)
- moved LED2 19.3 mm to (50.4, 92.0), turned to 90 degrees
- moved D1 18.9 mm to (53.4, 85.3)
- moved U1 18.6 mm to (48.7, 85.1)
- moved LED1 18.2 mm to (47.3, 92.0)
- moved R10 14.8 mm to (53.5, 92.0)
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Connections:
- LCD1 pad 0: (no net) -> Net-(LCD1-Pad0)
- LCD1 pad 28: (no net) -> Net-(LCD1-Pad28)
- SW5 pad 3: (no net) -> Net-(SW5-Pad3)
- SW7 pad 3: (no net) -> Net-(SW7-Pad3)
- U3 pad 2: (no net) -> Net-(U3-Pad2)
Routing:
- net GND: track 0.00 -> 483.4 mm, vias 0 -> 15
- net +3V3: track 0.00 -> 219.4 mm, vias 0 -> 3
- net +5C: track 0.00 -> 166.9 mm, vias 0 -> 2
- net Net-(P3-Pad5): track 0.00 -> 127.4 mm
- net /MOSI: track 0.00 -> 121.5 mm, vias 0 -> 1
- net /MISO: track 0.00 -> 115.1 mm, vias 0 -> 1
- net /SCK: track 0.00 -> 108.0 mm, vias 0 -> 1
- net /D-: track 0.00 -> 81.7 mm
- net /D+: track 0.00 -> 81.5 mm
- net Net-(SW4-Pad1): track 0.00 -> 72.0 mm, vias 0 -> 1
- net Net-(P2-Pad2): track 0.00 -> 65.9 mm
- net /BATADC: track 0.00 -> 60.7 mm, vias 0 -> 3
- net /BUZZER: track 0.00 -> 60.7 mm, vias 0 -> 2
- net +BATT: track 0.00 -> 56.9 mm, vias 0 -> 2
- net /SCL: track 0.00 -> 53.9 mm, vias 0 -> 1
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- added copper zone on B.Cu, net GND
- added copper zone on F.Cu, net GND
Other:
- outline, holes or cut-outs redrawn
- net class Default: trace_width 0.25 -> 0.6
- board text added: "Backlight"
- board text added: "https://github.com/szdiy/LCD7th"
