File: hardware/LCD7th.sch (KiCad schematic (older format))
At the start: 58 parts, among them P1 USB_B, P2 BATT, P3 ICSP, P4 UART, P5 I2C, P6 5VCONN, P7 BATT, P8 BATT, SW1 SW1, SW2 SW2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

Commit message: update
Parts:
- C1, C10, C11, C12, C13, C14, C15, C16, C17, C18, C19, C2, C20, C21, C3, C4, C5, C6, C7, C8, C9: footprint Capacitors_SMD:C_0805_HandSoldering -> Capacitors_SMD:C_0603_HandSoldering
- D1: value B340A -> M7; footprint LCD7th:B340A -> LCD7th:DIODE_DO214AC-SMA
- D2, D3, LED1, LED2: footprint LEDs:LED_0805 -> LEDs:LED_0603
- D4: footprint Capacitors_SMD:C_0805_HandSoldering -> LEDs:LED_0603
- P8: footprint LCD7th:LiConn -> SmartEye:CR2477_s
- R1, R10, R12, R2, R3, R4, R5, R6, R7, R9: footprint Resistors_SMD:R_0805_HandSoldering -> Resistors_SMD:R_0603_HandSoldering
- SP1: footprint LCD7th:TAT-BP1109S -> Buzzers_Beepers:BUZZER
- X1: footprint Crystals:Crystal_SMD_5032_4Pads -> Crystals:crystal_FA238-TSX3225
Connections:
- no-connect marks 7 -> 6

Commit message: uppdate layout
Parts:
- D4: footprint LEDs:LED_0603 -> Connectors:CONN_2.54mm_1x2
- P4, P5: footprint Pin_Headers:Pin_Header_Straight_1x04 -> Connectors:CONN_2.54mm_1x4
- P6: footprint Pin_Headers:Pin_Header_Straight_1x02 -> Connectors:CONN_2.54mm_1x2
Changed lines of the file:
@@
 F 0 "D4" H 6725 6150 50  0000 C CNN
 F 1 "LED" H 6725 5950 50  0000 C CNN
-F 2 "LEDs:LED_0603" H 6725 6050 50  0001 C CNN
+F 2 "Connectors:CONN_2.54mm_1x2" H 6725 6050 50  0001 C CNN
 F 3 "" H 6725 6050 50  0000 C CNN
 	1    6725 6050
@@
 F 0 "P4" H 10525 2350 50  0000 C CNN
 F 1 "UART" V 10625 2100 50  0000 C CNN
-F 2 "Pin_Headers:Pin_Header_Straight_1x04" H 10525 2100 50  0001 C CNN
+F 2 "Connectors:CONN_2.54mm_1x4" H 10525 2100 50  0001 C CNN
 F 3 "" H 10525 2100 50  0000 C CNN
 	1    10525 2100
@@
 F 0 "P5" H 10525 3175 50  0000 C CNN
 F 1 "I2C" V 10625 2925 50  0000 C CNN
-F 2 "Pin_Headers:Pin_Header_Straight_1x04" H 10525 2925 50  0001 C CNN
+F 2 "Connectors:CONN_2.54mm_1x4" H 10525 2925 50  0001 C CNN
 F 3 "" H 10525 2925 50  0000 C CNN
 	1    10525 2925
@@
 F 0 "P6" H 10525 4625 50  0000 C CNN
 F 1 "5VCONN" V 10625 4475 50  0000 C CNN
-F 2 "Pin_Headers:Pin_Header_Straight_1x02" H 10525 4475 50  0001 C CNN
+F 2 "Connectors:CONN_2.54mm_1x2" H 10525 4475 50  0001 C CNN
 F 3 "" H 10525 4475 50  0000 C CNN
 	1    10525 4475
